Commit message: Update project files

File: bicycle_sim/urdf/racecar.urdf (robot description, URDF)
Before this commit: robot racecar, 8 links, 7 joints
Links:
- link ego_racecar/back_left_wheel: geometry visual cylinder length=0.3 radius=0.5
- link ego_racecar/back_right_wheel: geometry visual cylinder length=0.3 radius=0.5
- link ego_racecar/base_link: geometry visual box size=1.25 0.8799999999999999 0.1
- link ego_racecar/front_left_wheel: geometry visual cylinder length=0.3 radius=0.5
- link ego_racecar/front_right_wheel: geometry visual cylinder length=0.3 radius=0.5
- link ego_racecar/laser_model: geometry visual cylinder length=0.05 radius=0.026
Joints:
- joint base_to_back_left_wheel: origin xyz=0 0.590000 0.500000 -> xyz=0 0.59 0.5
- joint base_to_back_right_wheel: origin xyz=0 -0.590000 0.500000 -> xyz=0 -0.59 0.5
- joint base_to_front_left_hinge: origin xyz=1.250000 0.590000 0.500000 -> xyz=1.25 0.59 0.5
- joint base_to_front_right_hinge: origin xyz=1.250000 -0.590000 0.500000 -> xyz=1.25 -0.59 0.5
- joint base_to_laser_model: origin xyz=0.275000 0 0.165000 -> xyz=0.275 0 0.165
